Commit message: Aula 13 Completed!

File: Aula12/p_jpedro_description/urdf/common_properties.xacro (robot description, xacro)
@@ -11,8 +11,8 @@
     <color rgba="0.4 0.4 0.4 1.0"/>
   </material>
-  <material name="blue">
+  <material name="Blue">
     <color rgba="0.0 0.0 0.8 1.0"/>
   </material>
-  <material name="green">
+  <material name="Green">
     <color rgba="0.0 0.8 0.0 1.0"/>
   </material>

File: Aula12/p_jpedro_description/urdf/p_jpedro.gazebo.xacro (robot description, xacro)
@@ -5,5 +5,6 @@
   <xacro:arg name="imu_visual"    default="false"/>
   <gazebo reference="base_link">
-    <material>Gazebo/Green</material>
+    <material>Gazebo/${player_color}</material>
+<!--        <material>Gazebo/Green</material>-->
   </gazebo>
   <gazebo reference="cylinder">
@@ -11,5 +12,6 @@
   </gazebo>
    <gazebo reference="sphere">
-    <material>Gazebo/Green</material>
+    <material>Gazebo/${player_color}</material>
+<!--         <material>Gazebo/Green</material>-->
   </gazebo>
   <gazebo reference="wheel_left_link">

File: Aula12/p_jpedro_description/urdf/p_jpedro.urdf.xacro (robot description, xacro)
@@ -1,6 +1,11 @@
 <?xml version="1.0" ?>
 <robot name="turtlebot3_waffle_pi" xmlns:xacro="http://ros.org/wiki/xacro">
+  <!--  Xacro Args-->
+  <xacro:arg name="player_color" default="Green"/>
+  <!--  Convert arg to property-->
+    <xacro:property name="player_color" value="$(arg player_color)"/>
+  <!--  Includes -->
   <xacro:include filename="$(find p_jpedro_description)/urdf/common_properties.xacro"/>
-  <xacro:include filename="$(find p_jpedro_description)/urdf/turtlebot3_waffle_pi.gazebo.xacro"/>
+  <xacro:include filename="p_jpedro.gazebo.xacro"/>
   <link name="base_footprint"/>
   <joint name="base_joint" type="fixed">
@@ -15,5 +20,6 @@
         <mesh filename="package://turtlebot3_description/meshes/bases/waffle_pi_base.stl" scale="0.001 0.001 0.001"/>
       </geometry>
-      <material name="sporting"/>
+      <material name="$(arg player_color)"/>
+<!--        <material name="Green"/>-->
     </visual>
     <collision>
@@ -43,5 +49,5 @@
         <mesh filename="package://turtlebot3_description/meshes/wheels/left_tire.stl" scale="0.001 0.001 0.001"/>
       </geometry>
-      <material name="sporting"/>
+      <material name="white"/>
     </visual>
     <collision>
@@ -71,5 +77,5 @@
         <mesh filename="package://turtlebot3_description/meshes/wheels/right_tire.stl" scale="0.001 0.001 0.001"/>
       </geometry>
-      <material name="dark"/>
+      <material name="white"/>
     </visual>
     <collision>
@@ -207,5 +213,6 @@
         <sphere radius="0.048"/>
       </geometry>
-      <material name="dark"/>
+      <material name="$(arg player_color)"/>
+<!--            <material name="Green"/>-->
     </visual>
   </link>
